File: DC_DC_Conv_test/DC_DC_Conv_test.kicad_sch (KiCad schematic)
At the start: 10 parts, among them J1 39301040

Commit message: update U1
Parts:
- renumbered VR1 to U1
Changed lines of the file:
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@@
 		(dnp no)
 		(fields_autoplaced yes)
-		(property "Reference" "VR1"
+		(property "Reference" "U1"
 			(at 151.13 78.74 0)
 			(effects
@@
 			(project ""
 				(path "/b4f10ad6-f5d8-4961-ab6d-fd678b503fb0"
-					(reference "VR1")
+					(reference "U1")
 					(unit 1)
 				)
